File: Hardware/PrototymV1_rx/PrototypV1_rx.sch (KiCad schematic (older format))
At the start: 76 parts, among them IC1 FS8205A, IC2 DW01A-G, IC3 MAX485CPA+, IC4 LD1117V33, IC5 STM32G051K8T6, IC6 TP4056, IC7 DS18B20, J1 PMS, J10 PROGRAM, J11 GND, J12 DS18B20, J13 VBAT+, J14 VBAT-, J15 VIN, J16 AHT15_TEST, J17 PMS_TEST, J18 HC12_TEST, J19 RS486_TEST, J2 AHT15, J20 GND, J21 GND, J23 GND, J3 PROGRAMATOR, J4 RS485, J5 , J6 HC12, J7 GND, J8 BATTERY, J9 SOLAR, SW1 SW_Push

Commit message: Ukończono
Parts:
- IC1: symbol FS8205A:FS8205A -> PrototypV1_rx-rescue:FS8205A-FS8205A
- IC2: symbol DW01A-G:DW01A-G -> PrototypV1_rx-rescue:DW01A-G-DW01A-G
- IC3: symbol MAX485CPA+:MAX485CPA+ -> PrototypV1_rx-rescue:MAX485CPA+-MAX485CPA+
- IC4: symbol LD1117V33:LD1117V33 -> PrototypV1_rx-rescue:LD1117V33-LD1117V33
- IC5: symbol STM32G051K8T6:STM32G051K8T6 -> PrototypV1_rx-rescue:STM32G051K8T6-STM32G051K8T6
- IC6: symbol TP4056:TP4056 -> PrototypV1_rx-rescue:TP4056-TP4056
Changed lines of the file:
@@
 $EndDescr
 $Comp
-L STM32G051K8T6:STM32G051K8T6 IC5
+L PrototypV1_rx-rescue:STM32G051K8T6-STM32G051K8T6 IC5
 U 1 1 62E71D51
 P 7850 4400
@@
 AHT15
 $Comp
-L MAX485CPA+:MAX485CPA+ IC3
+L PrototypV1_rx-rescue:MAX485CPA+-MAX485CPA+ IC3
 U 1 1 62E78EEF
 P 3700 950
@@
 HC12
 $Comp
-L TP4056:TP4056 IC6
+L PrototypV1_rx-rescue:TP4056-TP4056 IC6
 U 1 1 62E7F8E0
 P 9000 800
@@
 TP4056
 $Comp
-L DW01A-G:DW01A-G IC2
+L PrototypV1_rx-rescue:DW01A-G-DW01A-G IC2
 U 1 1 62E84B66
 P 1800 3250
@@
 	1600 2250 1600 2000
 $Comp
-L FS8205A:FS8205A IC1
+L PrototypV1_rx-rescue:FS8205A-FS8205A IC1
 U 1 1 62E8981E
 P 1300 3900
@@
 BATTERY PROTECTION
 $Comp
-L LD1117V33:LD1117V33 IC4
+L PrototypV1_rx-rescue:LD1117V33-LD1117V33 IC4
 U 1 1 62E9A305
 P 5000 2000
